Commit message: modified urdf and params for esa_robot

File: examples/utils/urdf/robot.urdf (robot description, URDF)
Before this commit: robot mirror666, 29 links, 28 joints
Links:
- removed link EEA_TCP_link
- removed link EEB_TCP_link
- removed link EEC_TCP_link
- added link A10_link, mass 3; collision cylinder length=0.2 radius=0.07; visual cylinder length=0.2 radius=0.07
- added link A7_link, mass 3.0; collision cylinder length=0.4 radius=0.07; visual cylinder length=0.4 radius=0.07
- added link A8_link, mass 1.5; collision mesh filename=package://esa_mirror/model_resources/meshes/simple/esa_elbo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 scale=0.001 0.001 0.001; visual mesh filename=package://esa_mirror/model_resources/meshes/simple/esa_elbo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 scale=0.001 0.001 0.001
- added link A9_link, mass 1.5; collision mesh filename=package://esa_mirror/model_resources/meshes/simple/esa_elbo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 scale=0.001 0.001 0.001; visual mesh filename=package://esa_mirror/model_resources/meshes/simple/esa_elbo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 scale=0.001 0.001 0.001
- added link A_TCP_link
- added link B10_link, mass 3; collision cylinder length=0.2 radius=0.07; visual cylinder length=0.2 radius=0.07
- added link B7_link, mass 3.0; collision cylinder length=0.4 radius=0.07; visual cylinder length=0.4 radius=0.07
- added link B8_link, mass 1.5; collision mesh filename=package://esa_mirror/model_resources/meshes/simple/esa_elbo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 scale=0.001 0.001 0.001; visual mesh filename=package://esa_mirror/model_resources/meshes/simple/esa_elbo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 scale=0.001 0.001 0.001
- added link B9_link, mass 1.5; collision mesh filename=package://esa_mirror/model_resources/meshes/simple/esa_elbo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 scale=0.001 0.001 0.001; visual mesh filename=package://esa_mirror/model_resources/meshes/simple/esa_elbo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 scale=0.001 0.001 0.001
- added link B_TCP_link
- added link C10_link, mass 3; collision cylinder length=0.2 radius=0.07; visual cylinder length=0.2 radius=0.07
- added link C7_link, mass 3.0; collision cylinder length=0.4 radius=0.07; visual cylinder length=0.4 radius=0.07
- added link C8_link, mass 1.5; collision mesh filename=package://esa_mirror/model_resources/meshes/simple/esa_elbo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 scale=0.001 0.001 0.001; visual mesh filename=package://esa_mirror/model_resources/meshes/simple/esa_elbo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 scale=0.001 0.001 0.001
- added link C9_link, mass 1.5; collision mesh filename=package://esa_mirror/model_resources/meshes/simple/esa_elbo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 scale=0.001 0.001 0.001; visual mesh filename=package://esa_mirror/model_resources/meshes/simple/esa_elbo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 scale=0.001 0.001 0.001
- added link C_TCP_link
- link A1_link: mass 5.0 -> 3.0; geometry collision cylinder length=0.4 radius=0.07; visual cylinder length=0.4 radius=0.07
- link A2_link: mass 3.5 -> 1.5; geometry collision mesh filename=package://esa_mirror/model_resources/meshes/simple/esa_elbo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 scale=0.001 0.001 0.001; visual mesh filename=package://esa_mirror/model_resources/meshes/simple/esa_elbo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 scale=0.001 0.001 0.001
- link A3_link: mass 2.5 -> 1.5; geometry collision mesh filename=package://esa_mirror/model_resources/meshes/simple/esa_elbo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 scale=0.001 0.001 0.001; visual mesh filename=package://esa_mirror/model_resources/meshes/simple/esa_elbo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 scale=0.001 0.001 0.001
- link A4_link: mass 4.4 -> 3.0; geometry collision cylinder length=0.4 radius=0.07; visual cylinder length=0.4 radius=0.07
- link A5_link: mass 2.9 -> 1.5; geometry collision mesh filename=package://esa_mirror/model_resources/meshes/simple/esa_elbo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 scale=0.001 0.001 0.001; visual mesh filename=package://esa_mirror/model_resources/meshes/simple/esa_elbo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 scale=0.001 0.001 0.001
- link A6_link: mass 2.0 -> 1.5; geometry collision mesh filename=package://esa_mirror/model_resources/meshes/simple/esa_elbo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 scale=0.001 0.001 0.001; visual mesh filename=package://esa_mirror/model_resources/meshes/simple/esa_elbo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 scale=0.001 0.001 0.001
- link B1_link: mass 5.0 -> 3.0; geometry collision cylinder length=0.4 radius=0.07; visual cylinder length=0.4 radius=0.07
- link B2_link: mass 3.5 -> 1.5; geometry collision mesh filename=package://esa_mirror/model_resources/meshes/simple/esa_elbo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 scale=0.001 0.001 0.001; visual mesh filename=package://esa_mirror/model_resources/meshes/simple/esa_elbo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 scale=0.001 0.001 0.001
- link B3_link: mass 2.5 -> 1.5; geometry collision mesh filename=package://esa_mirror/model_resources/meshes/simple/esa_elbo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 scale=0.001 0.001 0.001; visual mesh filename=package://esa_mirror/model_resources/meshes/simple/esa_elbo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 scale=0.001 0.001 0.001
- link B4_link: mass 4.4 -> 3.0; geometry collision cylinder length=0.4 radius=0.07; visual cylinder length=0.4 radius=0.07
- link B5_link: mass 2.9 -> 1.5; geometry collision mesh filename=package://esa_mirror/model_resources/meshes/simple/esa_elbo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 scale=0.001 0.001 0.001; visual mesh filename=package://esa_mirror/model_resources/meshes/simple/esa_elbo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 scale=0.001 0.001 0.001
- link B6_link: mass 2.0 -> 1.5; geometry collision mesh filename=package://esa_mirror/model_resources/meshes/simple/esa_elbo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 scale=0.001 0.001 0.001; visual mesh filename=package://esa_mirror/model_resources/meshes/simple/esa_elbo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 scale=0.001 0.001 0.001
- link C1_link: mass 5.0 -> 3.0; geometry collision cylinder length=0.4 radius=0.07; visual cylinder length=0.4 radius=0.07
- link C2_link: mass 3.5 -> 1.5; geometry collision mesh filename=package://esa_mirror/model_resources/meshes/simple/esa_elbo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 scale=0.001 0.001 0.001; visual mesh filename=package://esa_mirror/model_resources/meshes/simple/esa_elbo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 scale=0.001 0.001 0.001
- link C3_link: mass 2.5 -> 1.5; geometry collision mesh filename=package://esa_mirror/model_resources/meshes/simple/esa_elbo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 scale=0.001 0.001 0.001; visual mesh filename=package://esa_mirror/model_resources/meshes/simple/esa_elbo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 scale=0.001 0.001 0.001
- link C4_link: mass 4.4 -> 3.0; geometry collision cylinder length=0.4 radius=0.07; visual cylinder length=0.4 radius=0.07
- link C5_link: mass 2.9 -> 1.5; geometry collision mesh filename=package://esa_mirror/model_resources/meshes/simple/esa_elbo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 scale=0.001 0.001 0.001; visual mesh filename=package://esa_mirror/model_resources/meshes/simple/esa_elbo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 scale=0.001 0.001 0.001
- link C6_link: mass 2.0 -> 1.5; geometry collision mesh filename=package://esa_mirror/model_resources/meshes/simple/esa_elbo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 scale=0.001 0.001 0.001; visual mesh filename=package://esa_mirror/model_resources/meshes/simple/esa_elbo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 scale=0.001 0.001 0.001
Joints:
- removed joint EEA_TCP_joint
- removed joint EEB_TCP_joint
- removed joint EEC_TCP_joint
- added joint A10_joint: type revolute, parent A9_link, child A10_link, origin xyz=0 -0.075 0.07 rpy=0 0 0, axis 0 0 1, limit lower=-6.283 upper=6.283 effort=200 velocity=12
- added joint A7_joint: type revolute, parent A6_link, child A7_link, origin xyz=0 -0.075 0.07 rpy=0 0 0, axis 0 0 1, limit lower=-6.283 upper=6.283 effort=200 velocity=12
- added joint A8_joint: type fixed, parent A7_link, child A8_link, origin xyz=0 0 0.4 rpy=0 0 0
- added joint A9_joint: type revolute, parent A8_link, child A9_link, origin xyz=0 -0.075 0.07 rpy=0 0 0, axis 0 1 0, limit lower=-3.1415 upper=3.1415 effort=200 velocity=12
- added joint A_TCP_joint: type fixed, parent EEA_link, child A_TCP_link, origin xyz=0.0 0.0 0.1 rpy=0 0 0
- added joint B10_joint: type revolute, parent B9_link, child B10_link, origin xyz=0 -0.075 0.07 rpy=0 0 0, axis 0 0 1, limit lower=-6.283 upper=6.283 effort=200 velocity=12
- added joint B7_joint: type revolute, parent B6_link, child B7_link, origin xyz=0 -0.075 0.07 rpy=0 0 0, axis 0 0 1, limit lower=-6.283 upper=6.283 effort=200 velocity=12
- added joint B8_joint: type fixed, parent B7_link, child B8_link, origin xyz=0 0 0.4 rpy=0 0 0
- added joint B9_joint: type revolute, parent B8_link, child B9_link, origin xyz=0 -0.075 0.07 rpy=0 0 0, axis 0 1 0, limit lower=-3.1415 upper=3.1415 effort=200 velocity=12
- added joint B_TCP_joint: type fixed, parent EEB_link, child B_TCP_link, origin xyz=0.0 0.0 0.1 rpy=0 0 0
- added joint C10_joint: type revolute, parent C9_link, child C10_link, origin xyz=0 -0.075 0.07 rpy=0 0 0, axis 0 0 1, limit lower=-6.283 upper=6.283 effort=200 velocity=12
- added joint C7_joint: type revolute, parent C6_link, child C7_link, origin xyz=0 -0.075 0.07 rpy=0 0 0, axis 0 0 1, limit lower=-6.283 upper=6.283 effort=200 velocity=12
- added joint C8_joint: type fixed, parent C7_link, child C8_link, origin xyz=0 0 0.4 rpy=0 0 0
- added joint C9_joint: type revolute, parent C8_link, child C9_link, origin xyz=0 -0.075 0.07 rpy=0 0 0, axis 0 1 0, limit lower=-3.1415 upper=3.1415 effort=200 velocity=12
- added joint C_TCP_joint: type fixed, parent EEC_link, child C_TCP_link, origin xyz=0.0 0.0 0.1 rpy=0 0 0
- joint A1_joint: limit lower=-3.1415 upper=3.1415 effort=200.0 velocity=12.0 -> lower=-6.283 upper=6.283 effort=200 velocity=12
- joint A2_joint: axis 0 1 0 -> (none); limit lower=-3.1415 upper=3.1415 effort=200.0 velocity=12.0 -> (none); origin xyz=0 0 0.35 rpy=0 0 0 -> xyz=0 0 0.4 rpy=0 0 0; type revolute -> fixed
- joint A3_joint: limit lower=-3.1415 upper=3.1415 effort=200.0 velocity=12.0 -> lower=-3.1415 upper=3.1415 effort=200 velocity=12; origin xyz=0 0 0.25 rpy=0 0 0 -> xyz=0 -0.075 0.07 rpy=0 0 0
- joint A4_joint: axis 0 0 1 -> (none); limit lower=-3.1415 upper=3.1415 effort=200.0 velocity=12.0 -> (none); origin xyz=0 0 0.3 rpy=0 0 0 -> xyz=0 -0.075 0.07 rpy=0 0 0; type revolute -> fixed
- joint A5_joint: axis 0 1 0 -> (none); limit lower=-3.1415 upper=3.1415 effort=200.0 velocity=12.0 -> (none); origin xyz=0 0 0.35 rpy=0 0 0 -> xyz=0 0 0.4 rpy=0 0 3.14159265359; type revolute -> fixed
- joint A6_joint: axis 0 0 1 -> 0 1 0; limit lower=-3.1415 upper=3.1415 effort=200.0 velocity=12.0 -> lower=-3.1415 upper=3.1415 effort=200 velocity=12; origin xyz=0 0 0.15 rpy=0 0 0 -> xyz=0 -0.075 0.07 rpy=0 0 0
- joint B1_joint: limit lower=-3.1415 upper=3.1415 effort=200.0 velocity=12.0 -> lower=-6.283 upper=6.283 effort=200 velocity=12
- joint B2_joint: axis 0 1 0 -> (none); limit lower=-3.1415 upper=3.1415 effort=200.0 velocity=12.0 -> (none); origin xyz=0 0 0.35 rpy=0 0 0 -> xyz=0 0 0.4 rpy=0 0 0; type revolute -> fixed
- joint B3_joint: limit lower=-3.1415 upper=3.1415 effort=200.0 velocity=12.0 -> lower=-3.1415 upper=3.1415 effort=200 velocity=12; origin xyz=0 0 0.25 rpy=0 0 0 -> xyz=0 -0.075 0.07 rpy=0 0 0
- joint B4_joint: axis 0 0 1 -> (none); limit lower=-3.1415 upper=3.1415 effort=200.0 velocity=12.0 -> (none); origin xyz=0 0 0.3 rpy=0 0 0 -> xyz=0 -0.075 0.07 rpy=0 0 0; type revolute -> fixed
- joint B5_joint: axis 0 1 0 -> (none); limit lower=-3.1415 upper=3.1415 effort=200.0 velocity=12.0 -> (none); origin xyz=0 0 0.35 rpy=0 0 0 -> xyz=0 0 0.4 rpy=0 0 3.14159265359; type revolute -> fixed
- joint B6_joint: axis 0 0 1 -> 0 1 0; limit lower=-3.1415 upper=3.1415 effort=200.0 velocity=12.0 -> lower=-3.1415 upper=3.1415 effort=200 velocity=12; origin xyz=0 0 0.15 rpy=0 0 0 -> xyz=0 -0.075 0.07 rpy=0 0 0
- joint C1_joint: limit lower=-3.1415 upper=3.1415 effort=200.0 velocity=12.0 -> lower=-6.283 upper=6.283 effort=200 velocity=12
- joint C2_joint: axis 0 1 0 -> (none); limit lower=-3.1415 upper=3.1415 effort=200.0 velocity=12.0 -> (none); origin xyz=0 0 0.35 rpy=0 0 0 -> xyz=0 0 0.4 rpy=0 0 0; type revolute -> fixed
- joint C3_joint: limit lower=-3.1415 upper=3.1415 effort=200.0 velocity=12.0 -> lower=-3.1415 upper=3.1415 effort=200 velocity=12; origin xyz=0 0 0.25 rpy=0 0 0 -> xyz=0 -0.075 0.07 rpy=0 0 0
- joint C4_joint: axis 0 0 1 -> (none); limit lower=-3.1415 upper=3.1415 effort=200.0 velocity=12.0 -> (none); origin xyz=0 0 0.3 rpy=0 0 0 -> xyz=0 -0.075 0.07 rpy=0 0 0; type revolute -> fixed
- joint C5_joint: axis 0 1 0 -> (none); limit lower=-3.1415 upper=3.1415 effort=200.0 velocity=12.0 -> (none); origin xyz=0 0 0.35 rpy=0 0 0 -> xyz=0 0 0.4 rpy=0 0 3.14159265359; type revolute -> fixed
- joint C6_joint: axis 0 0 1 -> 0 1 0; limit lower=-3.1415 upper=3.1415 effort=200.0 velocity=12.0 -> lower=-3.1415 upper=3.1415 effort=200 velocity=12; origin xyz=0 0 0.15 rpy=0 0 0 -> xyz=0 -0.075 0.07 rpy=0 0 0
- joint EEA_joint: origin xyz=0 0 0.3 rpy=0 0 0 -> xyz=0 0 0.2 rpy=0 0 0; parent A6_link -> A10_link
- joint EEB_joint: origin xyz=0 0 0.3 rpy=0 0 0 -> xyz=0 0 0.2 rpy=0 0 0; parent B6_link -> B10_link
- joint EEC_joint: origin xyz=0 0 0.3 rpy=0 0 0 -> xyz=0 0 0.2 rpy=0 0 0; parent C6_link -> C10_link
