Commit message: Ready for simulation

File: examples/utils/urdf/centauro.urdf (robot description, URDF)
Before this commit: robot centauro, 75 links, 74 joints
Joints:
- joint torso_yaw: limit lower=-2.618 upper=2.618 effort=147 velocity=5.7 -> lower=-1.5 upper=1.5 effort=147 velocity=5.7

Commit message: minor changes

File: examples/utils/urdf/centauro.urdf (robot description, URDF)
Before this commit: robot centauro, 75 links, 74 joints
Links:
- link LElb: geometry collision mesh filename=package://cogimon_urdf/meshes/simple/Elbow.STL scale=0.0011 -0.0011 0.0011; visual mesh filename=package://cogimon_urdf/meshes/Elbow.STL scale=0.001 -0.001 0.001
- link LForearm: geometry collision mesh filename=package://cogimon_urdf/meshes/simple/Forearm.STL scale=0.0011 -0.0011 0.0011; visual mesh filename=package://cogimon_urdf/meshes/Forearm.STL scale=0.001 -0.001 0.001
- link LShp: geometry collision mesh filename=package://cogimon_urdf/meshes/simple/ShoulderPitch.STL scale=0.0011 -0.0011 0.0011; visual mesh filename=package://cogimon_urdf/meshes/ShoulderPitch.STL scale=0.001 -0.001 0.001
- link LShr: geometry collision mesh filename=package://cogimon_urdf/meshes/simple/ShoulderRoll.STL scale=0.0011 -0.0011 0.0011; visual mesh filename=package://cogimon_urdf/meshes/ShoulderRoll.STL scale=0.001 -0.001 0.001
- link LShy: geometry collision mesh filename=package://cogimon_urdf/meshes/simple/ShoulderYaw.STL scale=0.0011 -0.0011 0.0011; visual mesh filename=package://cogimon_urdf/meshes/ShoulderYaw.STL scale=0.001 -0.001 0.001
- link LWrMot2: geometry collision mesh filename=package://cogimon_urdf/meshes/simple/ForearmPitch.STL scale=0.0011 -0.0011 0.0011; visual mesh filename=package://cogimon_urdf/meshes/ForearmPitch.STL scale=0.001 -0.001 0.001
- link LWrMot3: geometry collision mesh filename=package://cogimon_urdf/meshes/simple/ForearmYaw.STL scale=0.0011 -0.0011 0.0011; visual mesh filename=package://cogimon_urdf/meshes/ForearmYaw.STL scale=0.001 -0.001 0.001
- link RElb: geometry collision mesh filename=package://cogimon_urdf/meshes/simple/Elbow.STL scale=0.001 0.0011 0.0011; visual mesh filename=package://cogimon_urdf/meshes/Elbow.STL scale=0.001 0.001 0.001
- link RForearm: geometry collision mesh filename=package://cogimon_urdf/meshes/simple/Forearm.STL scale=0.0011 0.0011 0.0011; visual mesh filename=package://cogimon_urdf/meshes/Forearm.STL scale=0.001 0.001 0.001
- link RShp: geometry collision mesh filename=package://cogimon_urdf/meshes/simple/ShoulderPitch.STL scale=0.0011 0.0011 0.0011; visual mesh filename=package://cogimon_urdf/meshes/ShoulderPitch.STL scale=0.001 0.001 0.001
- link RShr: geometry collision mesh filename=package://cogimon_urdf/meshes/simple/ShoulderRoll.STL scale=0.0011 0.0011 0.0011; visual mesh filename=package://cogimon_urdf/meshes/ShoulderRoll.STL scale=0.001 0.001 0.001
- link RShy: geometry collision mesh filename=package://cogimon_urdf/meshes/simple/ShoulderYaw.STL scale=0.0011 0.0011 0.0011; visual mesh filename=package://cogimon_urdf/meshes/ShoulderYaw.STL scale=0.001 0.001 0.001
- link RWrMot2: geometry collision mesh filename=package://cogimon_urdf/meshes/simple/ForearmPitch.STL scale=0.0011 0.0011 0.0011; visual mesh filename=package://cogimon_urdf/meshes/ForearmPitch.STL scale=0.001 0.001 0.001
- link RWrMot3: geometry collision mesh filename=package://cogimon_urdf/meshes/simple/ForearmYaw.STL scale=0.0011 0.0011 0.0011; visual mesh filename=package://cogimon_urdf/meshes/ForearmYaw.STL scale=0.001 0.001 0.001
- link ee1: geometry collision sphere radius=0.08; visual sphere radius=0.07
- link ee2: geometry collision sphere radius=0.08; visual sphere radius=0.07
- link knee_1: geometry collision mesh filename=package://centauro/centauro_urdf/meshes/convex_hull/knee.stl scale=0.0012 0.0012 0.0012; visual mesh filename=package://centauro/centauro_urdf/meshes/simplified/knee.stl scale=0.001 0.001 0.001
- link knee_2: geometry collision mesh filename=package://centauro/centauro_urdf/meshes/convex_hull/knee.stl scale=0.0012 0.0012 0.0012; visual mesh filename=package://centauro/centauro_urdf/meshes/simplified/knee.stl scale=0.001 0.001 0.001
- link l_wrist: geometry collision mesh filename=package://cogimon_urdf/meshes/simple/Wrist.STL scale=0.0011 -0.0011 0.0011; visual mesh filename=package://cogimon_urdf/meshes/Wrist.STL scale=0.001 -0.001 0.001
- link pelvis: geometry collision mesh filename=package://centauro/centauro_urdf/meshes/convex_hull/pelvis.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 scale=0.0011 0.0011 0.0011; visual mesh filename=package://centauro/centauro_urdf/meshes/simplified/pelvis.s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 scale=0.001 0.001 0.001
- link r_wrist: geometry collision mesh filename=package://cogimon_urdf/meshes/simple/Wrist.STL scale=0.0011 0.0011 0.0011; visual mesh filename=package://cogimon_urdf/meshes/Wrist.STL scale=0.001 0.001 0.001

Commit message: last fix

File: examples/utils/urdf/centauro.urdf (robot description, URDF)
Before this commit: robot centauro, 75 links, 74 joints
Links:
- link knee_1: geometry collision mesh filename=package://centauro/centauro_urdf/meshes/convex_hull/knee.stl scale=0.0013 0.0013 0.0013; visual mesh filename=package://centauro/centauro_urdf/meshes/simplified/knee.stl scale=0.001 0.001 0.001
- link knee_2: geometry collision mesh filename=package://centauro/centauro_urdf/meshes/convex_hull/knee.stl scale=0.0013 0.0013 0.0013; visual mesh filename=package://centauro/centauro_urdf/meshes/simplified/knee.stl scale=0.001 0.001 0.001
- link knee_3: geometry collision mesh filename=package://centauro/centauro_urdf/meshes/convex_hull/knee.stl scale=0.0013 0.0013 0.0013; visual mesh filename=package://centauro/centauro_urdf/meshes/simplified/knee.stl scale=0.001 0.001 0.001
- link knee_4: geometry collision mesh filename=package://centauro/centauro_urdf/meshes/convex_hull/knee.stl scale=0.0013 0.0013 0.0013; visual mesh filename=package://centauro/centauro_urdf/meshes/simplified/knee.stl scale=0.001 0.001 0.001

Commit message: fixed interpolator for ankle_yaws

File: examples/utils/urdf/centauro.urdf (robot description, URDF)
Before this commit: robot centauro, 75 links, 74 joints
Links:
- link LElb: geometry collision mesh filename=package://cogimon_urdf/meshes/simple/Elbow.STL scale=0.0012 -0.0012 0.0012; visual mesh filename=package://cogimon_urdf/meshes/Elbow.STL scale=0.001 -0.001 0.001
- link LForearm: geometry collision mesh filename=package://cogimon_urdf/meshes/simple/Forearm.STL scale=0.0012 -0.0012 0.0012; visual mesh filename=package://cogimon_urdf/meshes/Forearm.STL scale=0.001 -0.001 0.001
- link LShp: geometry collision mesh filename=package://cogimon_urdf/meshes/simple/ShoulderPitch.STL scale=0.0012 -0.0012 0.0012; visual mesh filename=package://cogimon_urdf/meshes/ShoulderPitch.STL scale=0.001 -0.001 0.001
- link LShr: geometry collision mesh filename=package://cogimon_urdf/meshes/simple/ShoulderRoll.STL scale=0.0012 -0.0012 0.0012; visual mesh filename=package://cogimon_urdf/meshes/ShoulderRoll.STL scale=0.001 -0.001 0.001
- link LShy: geometry collision mesh filename=package://cogimon_urdf/meshes/simple/ShoulderYaw.STL scale=0.0012 -0.0012 0.0012; visual mesh filename=package://cogimon_urdf/meshes/ShoulderYaw.STL scale=0.001 -0.001 0.001
- link LWrMot2: geometry collision mesh filename=package://cogimon_urdf/meshes/simple/ForearmPitch.STL scale=0.0012 -0.0012 0.0012; visual mesh filename=package://cogimon_urdf/meshes/ForearmPitch.STL scale=0.001 -0.001 0.001
- link LWrMot3: geometry collision mesh filename=package://cogimon_urdf/meshes/simple/ForearmYaw.STL scale=0.0012 -0.0012 0.0012; visual mesh filename=package://cogimon_urdf/meshes/ForearmYaw.STL scale=0.001 -0.001 0.001
- link RElb: geometry collision mesh filename=package://cogimon_urdf/meshes/simple/Elbow.STL scale=0.0012 0.0012 0.0012; visual mesh filename=package://cogimon_urdf/meshes/Elbow.STL scale=0.001 0.001 0.001
- link RForearm: geometry collision mesh filename=package://cogimon_urdf/meshes/simple/Forearm.STL scale=0.0012 0.0012 0.0012; visual mesh filename=package://cogimon_urdf/meshes/Forearm.STL scale=0.001 0.001 0.001
- link RShr: geometry collision mesh filename=package://cogimon_urdf/meshes/simple/ShoulderRoll.STL scale=0.0012 0.0012 0.0012; visual mesh filename=package://cogimon_urdf/meshes/ShoulderRoll.STL scale=0.001 0.001 0.001
- link RShy: geometry collision mesh filename=package://cogimon_urdf/meshes/simple/ShoulderYaw.STL scale=0.0012 0.0012 0.0012; visual mesh filename=package://cogimon_urdf/meshes/ShoulderYaw.STL scale=0.001 0.001 0.001
- link RWrMot2: geometry collision mesh filename=package://cogimon_urdf/meshes/simple/ForearmPitch.STL scale=0.0012 0.0012 0.0012; visual mesh filename=package://cogimon_urdf/meshes/ForearmPitch.STL scale=0.001 0.001 0.001
- link RWrMot3: geometry collision mesh filename=package://cogimon_urdf/meshes/simple/ForearmYaw.STL scale=0.0012 0.0012 0.0012; visual mesh filename=package://cogimon_urdf/meshes/ForearmYaw.STL scale=0.001 0.001 0.001
- link ee1: geometry collision sphere radius=0.085; visual sphere radius=0.07
- link ee2: geometry collision sphere radius=0.085; visual sphere radius=0.07
- link l_wrist: geometry collision mesh filename=package://cogimon_urdf/meshes/simple/Wrist.STL scale=0.0012 -0.0012 0.0012; visual mesh filename=package://cogimon_urdf/meshes/Wrist.STL scale=0.001 -0.001 0.001
- link r_wrist: geometry collision mesh filename=package://cogimon_urdf/meshes/simple/Wrist.STL scale=0.0012 0.0012 0.0012; visual mesh filename=package://cogimon_urdf/meshes/Wrist.STL scale=0.001 0.001 0.001
