Commit message: some fix and updated urdf and srdf to latest centauro version

File: examples/utils/urdf/centauro.urdf (robot description, URDF)
Before this commit: robot centauro, 75 links, 74 joints
Links:
- removed link DWYTorso
- removed link LElb
- removed link LForearm
- removed link LShp
- removed link LShr
- removed link LShy
- removed link LWrMot2
- removed link LWrMot3
- removed link RElb
- removed link RForearm
- removed link RShp
- removed link RShr
- removed link RShy
- removed link RWrMot2
- removed link RWrMot3
- removed link arm1_7
- removed link arm2_7
- removed link camera_central
- removed link camera_left
- removed link camera_right
- removed link ee1
- removed link ee2
- removed link kinect
- removed link kinect2_rgb_frame
- removed link kinect2_rgb_optical_frame
- removed link l_wrist
- removed link neck_2
- removed link neck_3
- removed link r_wrist
- removed link velodyne_mount
- added link D435_head_camera_bottom_screw_frame
- added link D435_head_camera_link, mass 0.564; collision box size=0.02505 0.09 0.025; visual mesh filename=package://centauro_urdf/meshes/realsense/d435.dae
- added link D435i_camera_bottom_screw_frame
- added link D435i_camera_link, mass 0.564; collision box size=0.02505 0.09 0.025; visual mesh filename=package://centauro_urdf/meshes/realsense/d435.dae
- added link ball1, mass 1.27; collision mesh filename=package://centauro_urdf/meshes/simple/BallHand.stl scale=0.001 0.001 0.001; visual mesh filename=package://centauro_urdf/meshes/BallHand.stl scale=0.001 0.001 0.001
- added link ball1_tip
- added link ball2, mass 1.27; collision mesh filename=package://centauro_urdf/meshes/simple/BallHand.stl scale=0.001 0.001 0.001; visual mesh filename=package://centauro_urdf/meshes/BallHand.stl scale=0.001 0.001 0.001
- added link ball2_tip
- added link base_link
- added link contact_1
- added link contact_2
- added link contact_3
- added link contact_4
- added link d435_head_motor, mass 0.33878686; collision mesh filename=package://centauro_urdf/meshes/simple/neck-pitch_mesh.stl scale=0.001 0.001 0.001; visual mesh filename=package://centauro_urdf/meshes/neck-pitch_mesh.stl scale=0.001 0.001 0.001
- added link velodyne_motor, mass 0.33878686; collision mesh filename=package://centauro_urdf/meshes/simple/lidar_mesh.stl scale=0.001 0.001 0.001; visual mesh filename=package://centauro_urdf/meshes/lidar_mesh.stl scale=0.001 0.001 0.001
- link ankle1_1: mass 1.2380744 -> 1.4023368; geometry collision mesh filename=package://centauro_urdf/meshes/v2/collision/ankle-pitch.stl scale=0.001 0.001 -0.001; visual mesh filename=package://centauro_urdf/meshes/v2/ankle-pitch.stl scale=0.001 0.001 -0.001
- link ankle1_2: mass 1.2380744 -> 1.4023368; geometry collision mesh filename=package://centauro_urdf/meshes/v2/collision/ankle-pitch.stl scale=0.001 0.001 0.001; visual mesh filename=package://centauro_urdf/meshes/v2/ankle-pitch.stl scale=0.001 0.001 0.001
- link ankle1_3: mass 1.2380744 -> 1.4023368; geometry collision mesh filename=package://centauro_urdf/meshes/v2/collision/ankle-pitch.stl scale=0.001 0.001 -0.001; visual mesh filename=package://centauro_urdf/meshes/v2/ankle-pitch.stl scale=0.001 0.001 -0.001
- link ankle1_4: mass 1.2380744 -> 1.4023368; geometry collision mesh filename=package://centauro_urdf/meshes/v2/collision/ankle-pitch.stl scale=0.001 0.001 0.001; visual mesh filename=package://centauro_urdf/meshes/v2/ankle-pitch.stl scale=0.001 0.001 0.001
- link ankle2_1: mass 1.1565926 -> 1.7656714; geometry collision mesh filename=package://centauro_urdf/meshes/v2/collision/ankle-yaw.stl scale=0.001 -0.001 0.001; visual mesh filename=package://centauro_urdf/meshes/v2/ankle-yaw.stl scale=0.001 -0.001 0.001
- link ankle2_2: mass 1.1565926 -> 1.7656714; geometry collision mesh filename=package://centauro_urdf/meshes/v2/collision/ankle-yaw.stl scale=0.001 0.001 0.001; visual mesh filename=package://centauro_urdf/meshes/v2/ankle-yaw.stl scale=0.001 0.001 0.001
- link ankle2_3: mass 1.1565926 -> 1.7656714; geometry collision mesh filename=package://centauro_urdf/meshes/v2/collision/ankle-yaw.stl scale=0.001 -0.001 0.001; visual mesh filename=package://centauro_urdf/meshes/v2/ankle-yaw.stl scale=0.001 -0.001 0.001
- link ankle2_4: mass 1.1565926 -> 1.7656714; geometry collision mesh filename=package://centauro_urdf/meshes/v2/collision/ankle-yaw.stl scale=0.001 0.001 0.001; visual mesh filename=package://centauro_urdf/meshes/v2/ankle-yaw.stl scale=0.001 0.001 0.001
- link arm1_1: mass None -> 1.9628675; geometry collision mesh filename=package://centauro_urdf/meshes/simple/ShoulderPitch.STL scale=0.001 -0.001 0.001; visual mesh filename=package://centauro_urdf/meshes/ShoulderPitch.STL scale=0.001 -0.001 0.001
- link arm1_2: mass None -> 1.8595811; geometry collision mesh filename=package://centauro_urdf/meshes/simple/ShoulderRoll.STL scale=0.001 -0.001 0.001; visual mesh filename=package://centauro_urdf/meshes/ShoulderRoll.STL scale=0.001 -0.001 0.001
- link arm1_3: mass None -> 1.6678109; geometry collision mesh filename=package://centauro_urdf/meshes/simple/ShoulderYaw.STL scale=0.001 -0.001 0.001; visual mesh filename=package://centauro_urdf/meshes/ShoulderYaw.STL scale=0.001 -0.001 0.001
- link arm1_4: mass None -> 1.3157289; geometry collision mesh filename=package://centauro_urdf/meshes/simple/Elbow.STL scale=0.001 -0.001 0.001; visual mesh filename=package://centauro_urdf/meshes/Elbow.STL scale=0.001 -0.001 0.001
- link arm1_5: mass None -> 1.4908547; geometry collision mesh filename=package://centauro_urdf/meshes/simple/Forearm.STL scale=0.001 -0.001 0.001; visual mesh filename=package://centauro_urdf/meshes/Forearm.STL scale=0.001 -0.001 0.001
- link arm1_6: mass None -> 1.1263612; geometry collision mesh filename=package://centauro_urdf/meshes/simple/wrist_pitch_right.stl scale=0.001 -0.001 0.001; visual mesh filename=package://centauro_urdf/meshes/wrist_pitch_right.stl scale=0.001 -0.001 0.001
- link arm1_8: mass None -> 0
- link arm2_1: mass None -> 1.9628675; geometry collision mesh filename=package://centauro_urdf/meshes/simple/ShoulderPitch.STL scale=0.001 0.001 0.001; visual mesh filename=package://centauro_urdf/meshes/ShoulderPitch.STL scale=0.001 0.001 0.001
- link arm2_2: mass None -> 1.8595811; geometry collision mesh filename=package://centauro_urdf/meshes/simple/ShoulderRoll.STL scale=0.001 0.001 0.001; visual mesh filename=package://centauro_urdf/meshes/ShoulderRoll.STL scale=0.001 0.001 0.001
- link arm2_3: mass None -> 1.6678109; geometry collision mesh filename=package://centauro_urdf/meshes/simple/ShoulderYaw.STL scale=0.001 0.001 0.001; visual mesh filename=package://centauro_urdf/meshes/ShoulderYaw.STL scale=0.001 0.001 0.001
- link arm2_4: mass None -> 1.3157289; geometry collision mesh filename=package://centauro_urdf/meshes/simple/Elbow.STL scale=0.001 0.001 0.001; visual mesh filename=package://centauro_urdf/meshes/Elbow.STL scale=0.001 0.001 0.001
- link arm2_5: mass None -> 1.4908547; geometry collision mesh filename=package://centauro_urdf/meshes/simple/Forearm.STL scale=0.001 0.001 0.001; visual mesh filename=package://centauro_urdf/meshes/Forearm.STL scale=0.001 0.001 0.001
- link arm2_6: mass None -> 1.1263612; geometry collision mesh filename=package://centauro_urdf/meshes/simple/wrist_pitch_right.stl scale=0.001 0.001 0.001; visual mesh filename=package://centauro_urdf/meshes/wrist_pitch_right.stl scale=0.001 0.001 0.001
- link arm2_8: mass None -> 0
- link hip1_1: mass 1.9194403 -> 2.3349153; geometry collision mesh filename=package://centauro_urdf/meshes/v2/collision/hip-yaw.stl scale=0.001 -0.001 0.001; visual mesh filename=package://centauro_urdf/meshes/v2/hip-yaw.stl scale=0.001 -0.001 0.001
- link hip1_2: mass 1.9194403 -> 2.3349153; geometry collision mesh filename=package://centauro_urdf/meshes/v2/collision/hip-yaw.stl scale=0.001 0.001 0.001; visual mesh filename=package://centauro_urdf/meshes/v2/hip-yaw.stl scale=0.001 0.001 0.001
- link hip1_3: mass 1.9194403 -> 2.3349153; geometry collision mesh filename=package://centauro_urdf/meshes/v2/collision/hip-yaw.stl scale=0.001 -0.001 0.001; visual mesh filename=package://centauro_urdf/meshes/v2/hip-yaw.stl scale=0.001 -0.001 0.001
- link hip1_4: mass 1.9194403 -> 2.3349153; geometry collision mesh filename=package://centauro_urdf/meshes/v2/collision/hip-yaw.stl scale=0.001 0.001 0.001; visual mesh filename=package://centauro_urdf/meshes/v2/hip-yaw.stl scale=0.001 0.001 0.001
- link hip2_1: mass 2.7264471 -> 3.4572118; geometry collision mesh filename=package://centauro_urdf/meshes/v2/collision/hip-pitch.stl scale=0.001 0.001 -0.001; visual mesh filename=package://centauro_urdf/meshes/v2/hip-pitch.stl scale=0.001 0.001 -0.001
- link hip2_2: mass 2.7264471 -> 3.4572118; geometry collision mesh filename=package://centauro_urdf/meshes/v2/collision/hip-pitch.stl scale=0.001 0.001 0.001; visual mesh filename=package://centauro_urdf/meshes/v2/hip-pitch.stl scale=0.001 0.001 0.001
- link hip2_3: mass 2.7264471 -> 3.4572118; geometry collision mesh filename=package://centauro_urdf/meshes/v2/collision/hip-pitch.stl scale=0.001 0.001 -0.001; visual mesh filename=package://centauro_urdf/meshes/v2/hip-pitch.stl scale=0.001 0.001 -0.001
- link hip2_4: mass 2.7264471 -> 3.4572118; geometry collision mesh filename=package://centauro_urdf/meshes/v2/collision/hip-pitch.stl scale=0.001 0.001 0.001; visual mesh filename=package://centauro_urdf/meshes/v2/hip-pitch.stl scale=0.001 0.001 0.001
- link imu_link: mass 0.0 -> None
- link knee_1: mass 1.9356754 -> 2.1199315; geometry collision mesh filename=package://centauro_urdf/meshes/v2/collision/knee.stl scale=0.001 0.001 -0.001; visual mesh filename=package://centauro_urdf/meshes/v2/knee.stl scale=0.001 0.001 -0.001
- link knee_2: mass 1.9356754 -> 2.1199315; geometry collision mesh filename=package://centauro_urdf/meshes/v2/collision/knee.stl scale=0.001 0.001 0.001; visual mesh filename=package://centauro_urdf/meshes/v2/knee.stl scale=0.001 0.001 0.001
- link knee_3: mass 1.9356754 -> 2.1199315; geometry collision mesh filename=package://centauro_urdf/meshes/v2/collision/knee.stl scale=0.001 0.001 -0.001; visual mesh filename=package://centauro_urdf/meshes/v2/knee.stl scale=0.001 0.001 -0.001
- link knee_4: mass 1.9356754 -> 2.1199315; geometry collision mesh filename=package://centauro_urdf/meshes/v2/collision/knee.stl scale=0.001 0.001 0.001; visual mesh filename=package://centauro_urdf/meshes/v2/knee.stl scale=0.001 0.001 0.001
- link neck_1: geometry collision mesh filename=package://centauro_urdf/meshes/simple/head-base_mesh.stl scale=0.001 0.001 0.001; visual mesh filename=package://centauro_urdf/meshes/head-base_mesh.stl scale=0.001 0.001 0.001
- link pelvis: mass 16.097574 -> 26.584529; geometry collision mesh filename=package://centauro_urdf/meshes/simple/pelvis.stl scale=0.001 0.001 0.001; visual mesh filename=package://centauro_urdf/meshes/v2/pelvis.stl scale=0.001 0.001 0.001
- link torso_2: mass 11.492689 -> 12.553731; geometry collision mesh filename=package://centauro_urdf/meshes/simple/link1_no_head.stl scale=0.001 0.001 0.001; visual mesh filename=package://centauro_urdf/meshes/link1_no_head.stl scale=0.001 0.001 0.001
- link wheel_1: mass 1.7289003 -> 1.11164; geometry collision cylinder length=0.11 radius=0.078; visual mesh filename=package://centauro_urdf/meshes/v2/wheel.stl scale=0.001 0.001 -0.001
- link wheel_2: mass 1.7289003 -> 1.11164; geometry collision cylinder length=0.11 radius=0.078; visual mesh filename=package://centauro_urdf/meshes/v2/wheel.stl scale=0.001 0.001 0.001
- link wheel_3: mass 1.7289003 -> 1.11164; geometry collision cylinder length=0.11 radius=0.078; visual mesh filename=package://centauro_urdf/meshes/v2/wheel.stl scale=0.001 0.001 -0.001
- link wheel_4: mass 1.7289003 -> 1.11164; geometry collision cylinder length=0.11 radius=0.078; visual mesh filename=package://centauro_urdf/meshes/v2/wheel.stl scale=0.001 0.001 0.001
Joints:
- removed joint j_arm1_7
- removed joint j_arm2_7
- removed joint j_camera_central
- removed joint j_camera_left
- removed joint j_camera_right
- removed joint j_kinect
- removed joint j_kinect2_rgb_frame
- removed joint j_kinect_optical_frame
- removed joint j_velodyne
- removed joint jee1
- removed joint jee2
- removed joint jf1
- removed joint jf10
- removed joint jf11
- removed joint jf12
- removed joint jf13
- removed joint jf14
- removed joint jf15
- removed joint jf16
- removed joint jf2
- removed joint jf3
- removed joint jf4
- removed joint jf5
- removed joint jf6
- removed joint jf7
- removed joint jf8
- removed joint jf9
- removed joint l_wrist_joint
- removed joint neck_pitch
- removed joint neck_velodyne
- removed joint neck_yaw
- removed joint r_wrist_joint
- removed joint torso_renaming
- added joint D435_head_camera_joint: type fixed, parent d435_head_motor, child D435_head_camera_bottom_screw_frame, origin xyz=0.03015 0 -0.0125 rpy=0 0 0
- added joint D435_head_camera_link_joint: type fixed, parent D435_head_camera_bottom_screw_frame, child D435_head_camera_link, origin xyz=0 0.0175 0.0125 rpy=0 0 0
- added joint D435i_camera_joint: type fixed, parent pelvis, child D435i_camera_bottom_screw_frame, origin xyz=0.272 0 0.084 rpy=0 0.54 0
- added joint D435i_camera_link_joint: type fixed, parent D435i_camera_bottom_screw_frame, child D435i_camera_link, origin xyz=0.053 0.0 -0.035 rpy=0 0.0050 -0.008
- added joint base_joint: type fixed, parent pelvis, child base_link, origin xyz=0 0 0 rpy=0 0 0
- added joint contact_joint_1: type fixed, parent ankle2_1, child contact_1, origin xyz=0 0 -0.176 rpy=0 0 0
- added joint contact_joint_2: type fixed, parent ankle2_2, child contact_2, origin xyz=0 0 -0.176 rpy=0 0 0
- added joint contact_joint_3: type fixed, parent ankle2_3, child contact_3, origin xyz=0 0 -0.176 rpy=0 0 0
- added joint contact_joint_4: type fixed, parent ankle2_4, child contact_4, origin xyz=0 0 -0.176 rpy=0 0 0
- added joint d435_head_joint: type revolute, parent neck_1, child d435_head_motor, origin xyz=0.06 0 0.1375 rpy=0 0 0, axis 0 -1 0, limit lower=-1.1 upper=1.1 effort=35 velocity=5.7
- added joint j_arm1_8: type fixed, parent arm1_6, child ball1, origin xyz=0. -0.05 -0.105 rpy=0. 0. 0.
- added joint j_arm2_8: type fixed, parent arm2_6, child ball2, origin xyz=0. 0.05 -0.105 rpy=0. 0. 0.
- added joint j_ball1_fixed: type fixed, parent ball1, child arm1_8
- added joint j_ball1_tip: type fixed, parent ball1, child ball1_tip, origin xyz=0 0 -0.07 rpy=0 0 0
- added joint j_ball2_fixed: type fixed, parent ball2, child arm2_8
- added joint j_ball2_tip: type fixed, parent ball2, child ball2_tip, origin xyz=0 0 -0.07 rpy=0 0 0
- added joint neck_base: type fixed, parent torso_2, child neck_1, origin xyz=0.0030637045 0.0061607221 0.158 rpy=0 0 0, axis 0 0 1
- added joint velodyne_joint: type revolute, parent neck_1, child velodyne_motor, origin xyz=0.0822724 0 0.242 rpy=0 0 0, axis 0 -1 0, limit lower=-1.1 upper=1.1 effort=35 velocity=5.7
- joint ankle_pitch_1: axis 0 0 1 -> 0 0 -1; limit lower=-2.61799388 upper=2.61799388 effort=147 velocity=8.1 -> lower=-2.4056 upper=2.3184 effort=147 velocity=8.1; origin xyz=0.2 0.0 -0.10015 rpy=3.14159265359 0.0 0.0 -> xyz=0.0 0.2 0.10015 rpy=3.14159265359 0.0 0.0
- joint ankle_pitch_2: limit lower=-2.61799388 upper=2.61799388 effort=147 velocity=8.1 -> lower=-2.3266 upper=2.3914 effort=147 velocity=8.1; origin xyz=0.2 0.0 -0.10015 rpy=3.14159265359 0.0 0.0 -> xyz=0.0 0.2 -0.10015 rpy=3.14159265359 0.0 0.0
- joint ankle_pitch_3: axis 0 0 1 -> 0 0 -1; limit lower=-2.61799388 upper=2.61799388 effort=147 velocity=8.1 -> lower=-2.4696 upper=2.4464 effort=147 velocity=8.1; origin xyz=0.2 0.0 -0.10015 rpy=3.14159265359 0.0 0.0 -> xyz=0.0 0.2 0.10015 rpy=3.14159265359 0.0 0.0
- joint ankle_pitch_4: limit lower=-2.61799388 upper=2.61799388 effort=147 velocity=8.1 -> lower=-2.3426 upper=2.3934 effort=147 velocity=8.1; origin xyz=0.2 0.0 -0.10015 rpy=3.14159265359 0.0 0.0 -> xyz=0.0 0.2 -0.10015 rpy=3.14159265359 0.0 0.0
- joint ankle_yaw_1: axis 0 0 1 -> 0 0 -1; limit lower=-2.5 upper=2.5 effort=35 velocity=20.0 -> lower=-2.5626 upper=2.5384 effort=35 velocity=20.0; origin xyz=0.0 0.0 0.0 rpy=1.57079632679 0.0 1.57079632679 -> xyz=0.0 -0.139 -0.00085 rpy=-1.57079632679 0.0 0.0
- joint ankle_yaw_2: axis 0 0 1 -> 0 0 -1; limit lower=-2.5 upper=2.5 effort=35 velocity=20.0 -> lower=-2.5546 upper=2.5484 effort=35 velocity=20.0; origin xyz=0.0 0.0 0.0 rpy=1.57079632679 0.0 1.57079632679 -> xyz=0.0 -0.139 0.00085 rpy=-1.57079632679 0.0 0.0
- joint ankle_yaw_3: axis 0 0 1 -> 0 0 -1; limit lower=-2.5 upper=2.5 effort=35 velocity=20.0 -> lower=-2.5606 upper=2.5454 effort=35 velocity=20.0; origin xyz=0.0 0.0 0.0 rpy=1.57079632679 0.0 1.57079632679 -> xyz=0.0 -0.139 -0.00085 rpy=-1.57079632679 0.0 0.0
- joint ankle_yaw_4: axis 0 0 1 -> 0 0 -1; limit lower=-2.5 upper=2.5 effort=35 velocity=20.0 -> lower=-2.6046 upper=2.5514 effort=35 velocity=20.0; origin xyz=0.0 0.0 0.0 rpy=1.57079632679 0.0 1.57079632679 -> xyz=0.0 -0.139 0.00085 rpy=-1.57079632679 0.0 0.0
- joint hip_pitch_1: axis 0 0 1 -> 0 0 -1; limit lower=-2.07 upper=2.07 effort=304 velocity=8.8 -> lower=-2.0226 upper=2.02748 effort=304 velocity=8.8; origin xyz=0.0 0.0 0.059 rpy=1.57079632679 0.0 0.50709869865 -> xyz=0.0 0.1146 -0.0625 rpy=1.57079632679 0.0 0.0
- joint hip_pitch_2: limit lower=-2.06 upper=2.09439510 effort=304 velocity=8.8 -> lower=-2.0156 upper=2.0354 effort=304 velocity=8.8; origin xyz=0.0 0.0 0.059 rpy=1.57079632679 0.0 2.63449395494 -> xyz=0.0 -0.1146 -0.0625 rpy=1.57079632679 0.0 0.0
- joint hip_pitch_3: axis 0 0 1 -> 0 0 -1; limit lower=-2.07 upper=2.09439510 effort=304 velocity=8.8 -> lower=-2.0126 upper=2.0384 effort=304 velocity=8.8; origin xyz=0.0 0.0 0.059 rpy=1.57079632679 0.0 2.63449395494 -> xyz=0.0 0.1146 -0.0625 rpy=1.57079632679 0.0 0.0
- joint hip_pitch_4: limit lower=-2.09439510 upper=2.09439510 effort=304 velocity=8.8 -> lower=-2.0326 upper=2.0524 effort=304 velocity=8.8; origin xyz=0.0 0.0 0.059 rpy=1.57079632679 0.0 0.50709869865 -> xyz=0.0 -0.1146 -0.0625 rpy=1.57079632679 0.0 0.0
- joint hip_yaw_1: axis 0 0 1 -> 0 0 -1; limit lower=-2.00 upper=2.48 effort=304 velocity=8.8 -> lower=-2.03 upper=2.51 effort=304 velocity=8.8; origin xyz=0.25 0.125 -0.0566 rpy=3.14159265359 0.0 0.50709869865 -> xyz=0.25 0.125 -0.0566 rpy=0.0 0.0 0.0
- joint hip_yaw_2: axis 0 0 1 -> 0 0 -1; limit lower=-2.48 upper=2.00 effort=304 velocity=8.8 -> lower=-2.51 upper=2.03 effort=304 velocity=8.8; origin xyz=0.25 -0.125 -0.0566 rpy=3.14159265359 0.0 -0.50709869865 -> xyz=0.25 -0.125 -0.0566 rpy=0.0 0.0 0.0
- joint hip_yaw_3: axis 0 0 1 -> 0 0 -1; limit lower=-2.48 upper=2.0 effort=304 velocity=8.8 -> lower=-2.51 upper=2.03 effort=304 velocity=8.8; origin xyz=-0.25 0.125 -0.0566 rpy=3.14159265359 0.0 2.63449395494 -> xyz=-0.25 0.125 -0.0566 rpy=0.0 0.0 0.0
- joint hip_yaw_4: axis 0 0 1 -> 0 0 -1; limit lower=-2.0 upper=2.48 effort=304 velocity=8.8 -> lower=-2.03 upper=2.51 effort=304 velocity=8.8; origin xyz=-0.25 -0.125 -0.0566 rpy=3.14159265359 0.0 3.64869135224 -> xyz=-0.25 -0.125 -0.0566 rpy=0.0 0.0 0.0
- joint j_arm1_1: child LShp -> arm1_1; limit lower=-3.352 upper=1.603 effort=140 velocity=6.283 -> lower=-3.312 upper=1.615 effort=147.0 velocity=3.86; origin xyz=0.0457475 0.169137 0.155126 rpy=0.174533 0 -0.5235988 -> xyz=0.0457475 0.169137 0.116626 rpy=0.174533 0.0 -0.5235988; parent DWYTorso -> torso_2
- joint j_arm1_2: child LShr -> arm1_2; limit lower=0.0 upper=3.517 effort=140 velocity=6.283 -> lower=0.02 upper=3.431 effort=147.0 velocity=3.86; origin xyz=-0.09015 0.062 0 rpy=-0.1745327 0 0 -> xyz=-0.09015 0.062 0.0 rpy=-0.1745327 0.0 0.0; parent LShp -> arm1_1
- joint j_arm1_3: child LShy -> arm1_3; limit lower=-2.55 upper=2.55 effort=120 velocity=6.283 -> lower=-2.552 upper=2.566 effort=147.0 velocity=6.06; origin xyz=0.09015 0 -0.21815 rpy=0 0 0 -> xyz=0.09015 0.0 -0.21815; parent LShr -> arm1_2
- joint j_arm1_4: child LElb -> arm1_4; limit lower=-2.492 upper=0.298 effort=120 velocity=6.283 -> lower=-2.465 upper=0.28 effort=147.0 velocity=6.06; origin xyz=0.045 0.05515 -0.074 rpy=0 0 0 -> xyz=0.045 0.05515 -0.074; parent LShy -> arm1_3
- joint j_arm1_5: child LForearm -> arm1_5; limit lower=-2.55 upper=2.55 effort=35 velocity=6.283 -> lower=-2.569 upper=2.562 effort=55.0 velocity=11.72; origin xyz=-0.015 -0.05515 -0.095 rpy=0 0 0 -> xyz=-0.015 -0.05515 -0.095; parent LElb -> arm1_4
- joint j_arm1_6: child LWrMot2 -> arm1_6; limit lower=-1.562 upper=1.478 effort=35 velocity=6.283 -> lower=-1.529 upper=1.509 effort=55.0 velocity=11.72; origin xyz=0 0.049 -0.156 rpy=0 0 0 -> xyz=0.0 0.049 -0.156; parent LForearm -> arm1_5
- joint j_arm2_1: child RShp -> arm2_1; limit lower=-3.359 upper=1.606 effort=140 velocity=6.283 -> lower=-3.3458 upper=1.6012 effort=147.0 velocity=3.86; origin xyz=0.0457475 -0.169137 0.155126 rpy=-0.174533 0 0.5235988 -> xyz=0.0457475 -0.169137 0.116626 rpy=-0.174533 0.0 0.5235988; parent DWYTorso -> torso_2
- joint j_arm2_2: child RShr -> arm2_2; limit lower=-3.43 upper=0.0 effort=140 velocity=6.283 -> lower=-3.4258 upper=-0.0138 effort=147.0 velocity=3.86; origin xyz=-0.09015 -0.062 0 rpy=0.1745327 0 0 -> xyz=-0.09015 -0.062 0.0 rpy=0.1745327 0.0 0.0; parent RShp -> arm2_1
- joint j_arm2_3: child RShy -> arm2_3; limit lower=-2.55 upper=2.55 effort=120 velocity=6.283 -> lower=-2.5614 upper=2.5606 effort=147.0 velocity=6.06; origin xyz=0.09015 0 -0.21815 rpy=0 0 0 -> xyz=0.09015 0.0 -0.21815; parent RShr -> arm2_2
- joint j_arm2_4: child RElb -> arm2_4; limit lower=-2.488 upper=0.292 effort=120 velocity=6.283 -> lower=-2.4794 upper=0.2886 effort=147.0 velocity=6.06; origin xyz=0.045 -0.05515 -0.074 rpy=0 0 0 -> xyz=0.045 -0.05515 -0.074; parent RShy -> arm2_3
- joint j_arm2_5: child RForearm -> arm2_5; limit lower=-2.55 upper=2.55 effort=35 velocity=6.283 -> lower=-2.5394 upper=2.5546 effort=55.0 velocity=11.72; origin xyz=-0.015 0.05515 -0.095 rpy=0 0 0 -> xyz=-0.015 0.05515 -0.095; parent RElb -> arm2_4
- joint j_arm2_6: child RWrMot2 -> arm2_6; limit lower=-1.542 upper=1.508 effort=35 velocity=6.283 -> lower=-1.5154 upper=1.5156 effort=55.0 velocity=11.72; origin xyz=0 -0.049 -0.156 rpy=0 0 0 -> xyz=0.0 -0.049 -0.156; parent RForearm -> arm2_5
- joint j_wheel_1: limit lower=-1000000000000000 upper=1000000000000000 effort=35 velocity=20.0 -> effort=35 velocity=20.0; origin xyz=0.0 0.00085 0.235 rpy=1.57079632679 0.0 0.0 -> xyz=0.0 -0.0 -0.09835 rpy=1.57079632679 0.0 0.0
- joint j_wheel_2: axis 0 0 -1 -> 0 0 1; limit lower=-1000000000000000 upper=1000000000000000 effort=35 velocity=20.0 -> effort=35 velocity=20.0; origin xyz=0.0 0.00085 0.235 rpy=1.57079632679 0.0 0.0 -> xyz=0.0 0.0 -0.09835 rpy=1.57079632679 0.0 0.0
- joint j_wheel_3: limit lower=-1000000000000000 upper=1000000000000000 effort=35 velocity=20.0 -> effort=35 velocity=20.0; origin xyz=0.0 0.00085 0.235 rpy=1.57079632679 0.0 0.0 -> xyz=0.0 -0.0 -0.09835 rpy=1.57079632679 0.0 0.0
- joint j_wheel_4: axis 0 0 -1 -> 0 0 1; limit lower=-1000000000000000 upper=1000000000000000 effort=35 velocity=20.0 -> effort=35 velocity=20.0; origin xyz=0.0 0.00085 0.235 rpy=1.57079632679 0.0 0.0 -> xyz=0.0 0.0 -0.09835 rpy=1.57079632679 0.0 0.0
- joint knee_pitch_1: axis 0 0 1 -> 0 0 -1; limit lower=-2.61799388 upper=2.61799388 effort=304 velocity=8.8 -> lower=-2.4056 upper=2.3994 effort=304 velocity=8.8; origin xyz=0.0 0.3 -0.0036 rpy=3.14159265359 0.0 1.57079632679 -> xyz=0.0 -0.3 0.1182 rpy=3.14159265359 0.0 0.0
- joint knee_pitch_2: limit lower=-2.61799388 upper=2.61799388 effort=304 velocity=8.8 -> lower=-2.4006 upper=2.4034 effort=304 velocity=8.8; origin xyz=0.0 0.3 -0.0036 rpy=3.14159265359 0.0 1.57079632679 -> xyz=0.0 -0.3 -0.1182 rpy=3.14159265359 0.0 0.0
- joint knee_pitch_3: axis 0 0 1 -> 0 0 -1; limit lower=-2.61799388 upper=2.61799388 effort=304 velocity=8.8 -> lower=-2.4056 upper=2.4064 effort=304 velocity=8.8; origin xyz=0.0 0.3 -0.0036 rpy=3.14159265359 0.0 1.57079632679 -> xyz=0.0 -0.3 0.1182 rpy=3.14159265359 0.0 0.0
- joint knee_pitch_4: limit lower=-2.61799388 upper=2.61799388 effort=304 velocity=8.8 -> lower=-2.4176 upper=2.3884 effort=304 velocity=8.8; origin xyz=0.0 0.3 -0.0036 rpy=3.14159265359 0.0 1.57079632679 -> xyz=0.0 -0.3 -0.1182 rpy=3.14159265359 0.0 0.0
- joint reference: origin xyz=0.0 0.0 0.93445 -> (none)
- joint torso_yaw: limit lower=-1.5 upper=1.5 effort=147 velocity=5.7 -> lower=-2.618 upper=2.618 effort=147 velocity=5.7
- joint velodyne_calib_base_mount_joint: origin xyz=0.032768 -0.01 0.048219 rpy=0 1.5709 -0.316519   -> xyz=-0.01 0.02 0.06 rpy=0.025 0.019 0; parent neck_3 -> velodyne_motor
